File: PCB/AllPixelMini.sch (KiCad schematic (older format))
At the start: 25 parts, among them CON1 ML_USB_MINI, CON2 BARREL_JACK, P1 CONN_1, P2 CONN_1, Q1 NPN, U1 ATMEGA16U4/32U4, Y1 16MHz

Commit message: tweaked mini layout
Parts:
- removed CON2: BARREL_JACK, symbol BARREL_JACK
- added JP3: PT_INPUT, SparkFun-1X04_LOCK, symbol M04LOCK
- added P3: CONN_2, symbol CONN_2
- JP1: value OUTPUT2 -> PT_OUTPUT
Connections:
- wire segments 67 -> 70
- no-connect marks 22 -> 23
Other:
- moved on the sheet: JP1
Changed lines of the file:
@@
 LIBS:SparkFun
 LIBS:w_connectors
+LIBS:AllPixelMini-cache
 EELAYER 27 0
 EELAYER END
@@
 Sheet 1 1
 Title ""
-Date "25 apr 2015"
+Date "1 may 2015"
 Rev ""
 Comp ""
@@
 NoConn ~ 4400 4250
 $Comp
-L +5V #PWR1
+L +5V #PWR01
 U 1 1 53D3C5A9
 P 6400 1300
-F 0 "#PWR1" H 6400 1390 20  0001 C CNN
+F 0 "#PWR01" H 6400 1390 20  0001 C CNN
 F 1 "+5V" H 6400 1390 30  0000 C CNN
 F 2 "" H 6400 1300 60  0000 C CNN
@@
 	6400 1300 6400 1350
 $Comp
-L GND #PWR2
+L GND #PWR02
 U 1 1 53D3C600
 P 6450 2150
-F 0 "#PWR2" H 6450 2150 30  0001 C CNN
+F 0 "#PWR02" H 6450 2150 30  0001 C CNN
 F 1 "GND" H 6450 2080 30  0001 C CNN
 F 2 "" H 6450 2150 60  0000 C CNN
@@
 Wire Wire Line
 	1600 1700 1700 1700
-$Comp
-L BARREL_JACK CON2
-U 1 1 553B1AAF
-P 7100 4950
-F 0 "CON2" H 7100 5200 60  0000 C CNN
-F 1 "BARREL_JACK" H 7100 4750 60  0000 C CNN
-F 2 "" H 7100 4950 60  0000 C CNN
-F 3 "" H 7100 4950 60  0000 C CNN
-	1    7100 4950
-	-1   0    0    1
-$EndComp
 $Comp
 L CP1 C5
@@
 L M04LOCK JP1
 U 1 1 553B1ACF
-P 7550 4300
-F 0 "JP1" H 7350 4630 50  0000 L BNN
-F 1 "OUTPUT2" H 7350 4000 50  0000 L BNN
-F 2 "SparkFun-1X04_LOCK" H 7550 4450 50  0001 C CNN
-F 3 "" H 7550 4300 60  0000 C CNN
-	1    7550 4300
+P 8150 4200
+F 0 "JP1" H 7950 4530 50  0000 L BNN
+F 1 "PT_OUTPUT" H 7950 3900 50  0000 L BNN
+F 2 "SparkFun-1X04_LOCK" H 8150 4350 50  0001 C CNN
+F 3 "" H 8150 4200 60  0000 C CNN
+	1    8150 4200
 	-1   0    0    1
 $EndComp
@@
 VJACK
 Wire Wire Line
-	6750 5050 6800 5050
-Wire Wire Line
-	6750 4850 6800 4850
-Wire Wire Line
-	6800 4750 6800 4950
-Wire Wire Line
 	6800 4750 6350 4750
-Connection ~ 6800 4850
-Wire Wire Line
-	6800 5050 6800 5150
 Wire Wire Line
 	6800 5150 6350 5150
@@
 Wire Wire Line
 	6500 3750 6500 3700
-Text GLabel 7300 4300 0    30   Input ~ 0
+Text GLabel 7900 4200 0    30   Input ~ 0
 DATA
-Text GLabel 7300 4400 0    30   Input ~ 0
+Text GLabel 7900 4300 0    30   Input ~ 0
 CLK
-Text GLabel 7300 4200 0    30   Input ~ 0
+Text GLabel 7900 4100 0    30   Input ~ 0
 VJACK
-Text GLabel 7300 4500 0    30   Input ~ 0
-GND
-Wire Wire Line
-	7300 4200 7350 4200
-Wire Wire Line
-	7350 4300 7300 4300
-Wire Wire Line
-	7300 4400 7350 4400
-Wire Wire Line
-	7350 4500 7300 4500
+Text GLabel 7900 4400 0    30   Input ~ 0
+GND
+Wire Wire Line
+	7900 4100 7950 4100
+Wire Wire Line
+	7950 4200 7900 4200
+Wire Wire Line
+	7900 4300 7950 4300
+Wire Wire Line
+	7950 4400 7900 4400
+$Comp
+L M04LOCK JP3
+U 1 1 5542B3DA
+P 8200 4950
+F 0 "JP3" H 8000 5280 50  0000 L BNN
+F 1 "PT_INPUT" H 8000 4650 50  0000 L BNN
+F 2 "SparkFun-1X04_LOCK" H 8200 5100 50  0001 C CNN
+F 3 "" H 8200 4950 60  0000 C CNN
+	1    8200 4950
+	-1   0    0    1
+$EndComp
+Text GLabel 7950 4950 0    30   Input ~ 0
+DATA
+Text GLabel 7950 5050 0    30   Input ~ 0
+CLK
+Text GLabel 7950 5150 0    30   Input ~ 0
+GND
+Wire Wire Line
+	8000 4950 7950 4950
+Wire Wire Line
+	7950 5050 8000 5050
+Wire Wire Line
+	8000 5150 7950 5150
+$Comp
+L CONN_2 P3
+U 1 1 5542B430
+P 7150 4950
+F 0 "P3" V 7100 4950 40  0000 C CNN
+F 1 "CONN_2" V 7200 4950 40  0000 C CNN
+F 2 "" H 7150 4950 60  0000 C CNN
+F 3 "" H 7150 4950 60  0000 C CNN
+	1    7150 4950
+	1    0    0    -1
+$EndComp
+Wire Wire Line
+	6800 4750 6800 4850
+Wire Wire Line
+	6800 4850 6750 4850
+Wire Wire Line
+	6750 5050 6800 5050
+Wire Wire Line
+	6800 5050 6800 5150
+NoConn ~ 8000 4850
 $EndSCHEMATC
